File: hardware/lightning-map.kicad_sch (KiCad schematic)
At the start: 543 parts, among them J1 Screw_Terminal_01x02, J2 Screw_Terminal_01x04, U1 IS31FL3731-QF, U2 IS31FL3731-QF, U3 IS31FL3731-QF, U4 IS31FL3731-QF

Commit message: started working on usb c + esp32 integration
Parts:
- removed J1: Screw_Terminal_01x02, TerminalBlock:TerminalBlock_bornier-2_P5.08mm, symbol Connector:Screw_Terminal_01x02
- added C17, C19: 4.7uF, symbol Device:C
- added C18: C, symbol Device:C
- added C20: 1uF, symbol Device:C
- added J3: USB_C_Receptacle_PowerOnly_6P, symbol Connector:USB_C_Receptacle_PowerOnly_6P
- added R10, R11, R9: R, symbol Device:R
- added U5: ESP32-S3-WROOM-1, RF_Module:ESP32-S3-WROOM-1, symbol RF_Module:ESP32-S3-WROOM-1
- added U6: ADM7172ACPZ-3.3-R7, CP-8-21_ADI, symbol 2025-01-03_13-23-46:ADM7172ACPZ-3.3-R7
Connections:
- net GND: now also C17.2, C18.2, C19.1, C20.1, J3.A12 (GND), J3.B12 (GND), J3.S1 (SHIELD), R10.2, R9.2, U5.1 (GND), U5.40 (GND), U5.41 (GND), U6.6 (GND), U6.9 (GND)
- net VCC renamed +3.3V
- net +3.3V: now also C19.2, R11.1, U5.2 (3V3), U6.1 (VOUT), U6.2 (VOUT), U6.3 (SENSE)
- new net: C18.1, U6.4 (SS)
- new net: J3.A5 (CC1), R9.1
- new net: C20.2, R11.2, U5.3 (EN)
- new net: J3.B5 (CC2), R10.1
- new net +5V: C17.1, J3.A9 (VBUS), J3.B9 (VBUS), U6.5 (EN), U6.7 (VIN), U6.8 (VIN)
- no-connect marks 0 -> 1
Other:
- moved on the sheet: C1, C10, C11, C12, C13, C14, C15, C16, C2, C3, C4, C5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
